Commit message: Fix xacro warnings on Kinetic.

File: am_description/urdf/automower.urdf.xacro (robot description, xacro)
@@ -8,17 +8,17 @@
   <!-- PROPERTY LIST -->
   <!--All units in m-kg-s-radians unit system -->
-  <property name="M_PI" value="3.1415926535897931" />
+  <xacro:property name="M_PI" value="3.1415926535897931" />
   <!-- Main Body-base -->
-  <property name="base_x_size" value="0.72" />
-  <property name="base_y_size" value="0.55" />
-  <property name="base_z_size" value="0.23" />
-  <property name="base_mass" value="15" /> <!-- in kg-->
-  <property name="base_z_origin_to_wheel_origin" value="-0.07" />
+  <xacro:property name="base_x_size" value="0.72" />
+  <xacro:property name="base_y_size" value="0.55" />
+  <xacro:property name="base_z_size" value="0.23" />
+  <xacro:property name="base_mass" value="15" /> <!-- in kg-->
+  <xacro:property name="base_z_origin_to_wheel_origin" value="-0.07" />
   <!--Inertial macros for the box and cylinder. Units are kg*m^2-->
-  <macro name="box_inertia" params="m x y z">
+  <xacro:macro name="box_inertia" params="m x y z">
     <inertia  ixx="${m*(y*y+z*z)/12}" ixy = "0" ixz = "0"
               iyy="${m*(x*x+z*z)/12}" iyz = "0"
               izz="${m*(x*x+z*z)/12}" />
-  </macro>
+  </xacro:macro>
   <!-- BASE-LINK -->
   <!--Actual body/chassis of the robot-->

File: am_description/urdf/swivel_wheel.urdf.xacro (robot description, xacro)
@@ -3,19 +3,19 @@
   <!-- Wheels -->
 <!--
-  <property name="wheel_radius" value="0.125" />
-  <property name="wheel_height" value="0.032" />
+  <xacro:property name="wheel_radius" value="0.125" />
+  <xacro:property name="wheel_height" value="0.032" />
 -->
-  <property name="wheel_mass" value="0.5" /> <!-- in kg-->
+  <xacro:property name="wheel_mass" value="0.5" /> <!-- in kg-->
 <!--
-  <property name="base_x_origin_to_wheel_origin" value="0.25" />
-  <property name="base_y_origin_to_wheel_origin" value="0.3" />
-  <property name="base_z_origin_to_wheel_origin" value="0.0" />
+  <xacro:property name="base_x_origin_to_wheel_origin" value="0.25" />
+  <xacro:property name="base_y_origin_to_wheel_origin" value="0.3" />
+  <xacro:property name="base_z_origin_to_wheel_origin" value="0.0" />
 -->
-  <macro name="cylinder_inertia" params="m r h">
+  <xacro:macro name="cylinder_inertia" params="m r h">
     <inertia  ixx="${m*(3*r*r+h*h)/12}" ixy = "0" ixz = "0"
               iyy="${m*(3*r*r+h*h)/12}" iyz = "0"
               izz="${m*r*r/2}" />
-  </macro>
-  <macro name = "swivel_arm" params="lr index l offset">
+  </xacro:macro>
+  <xacro:macro name = "swivel_arm" params="lr index l offset">
     <link name="sw_arm_${lr}_${index}">
       <inertial>
@@ -34,5 +34,5 @@
       </visual>
     </link>
-  </macro>
+  </xacro:macro>
   <xacro:macro name="swivel_wheel" params="fb lr parent translateX translateY translateZ wheel_radius wheel_height flip"> <!--fb : front, back ; lr: left, right -->
     <!-- First link connected to parent-->

File: am_description/urdf/wheel.urdf.xacro (robot description, xacro)
@@ -3,18 +3,18 @@
   <!-- Wheels -->
 <!--
-  <property name="wheel_radius" value="0.125" />
-  <property name="wheel_height" value="0.032" />
+  <xacro:property name="wheel_radius" value="0.125" />
+  <xacro:property name="wheel_height" value="0.032" />
 -->
-  <property name="wheel_mass" value="0.3" /> <!-- in kg-->
+  <xacro:property name="wheel_mass" value="0.3" /> <!-- in kg-->
 <!--
-  <property name="base_x_origin_to_wheel_origin" value="0.25" />
-  <property name="base_y_origin_to_wheel_origin" value="0.3" />
-  <property name="base_z_origin_to_wheel_origin" value="0.0" />
+  <xacro:property name="base_x_origin_to_wheel_origin" value="0.25" />
+  <xacro:property name="base_y_origin_to_wheel_origin" value="0.3" />
+  <xacro:property name="base_z_origin_to_wheel_origin" value="0.0" />
 -->
-  <macro name="cylinder_inertia" params="m r h">
+  <xacro:macro name="cylinder_inertia" params="m r h">
     <inertia  ixx="${m*(3*r*r+h*h)/12}" ixy = "0" ixz = "0"
               iyy="${m*(3*r*r+h*h)/12}" iyz = "0"
               izz="${m*r*r/2}" />
-  </macro>
+  </xacro:macro>
   <xacro:macro name="wheel" params="fb lr parent translateX translateY translateZ wheel_radius wheel_height flip"> <!--fb : front, back ; lr: left, right -->
     <link name="${fb}_${lr}_wheel">
