Commit message: Fix inconsistent indentation & formatting in xacro files.

File: am_description/urdf/automower.urdf.xacro (robot description, xacro)
@@ -17,7 +17,7 @@
   <!--Inertial macros for the box and cylinder. Units are kg*m^2-->
   <xacro:macro name="box_inertia" params="m x y z">
-    <inertia  ixx="${m*(y*y+z*z)/12}" ixy = "0" ixz = "0"
-              iyy="${m*(x*x+z*z)/12}" iyz = "0"
-              izz="${m*(x*x+z*z)/12}" />
+    <inertia ixx="${m*(y*y+z*z)/12}" ixy="0" ixz="0"
+             iyy="${m*(x*x+z*z)/12}" iyz="0"
+             izz="${m*(x*x+z*z)/12}" />
   </xacro:macro>
   <!-- BASE-LINK -->
@@ -29,11 +29,11 @@
       <!--The 3x3 rotational inertia matrix. -->
       <!--<box_inertia  m="${base_mass}" x="${base_x_size}" y="${base_y_size}" z="${base_z_size}"/>-->
-      <box_inertia  m="${5*base_mass}" x="${base_x_size}" y="${base_y_size}" z="${base_z_size}"/>
+      <box_inertia m="${5*base_mass}" x="${base_x_size}" y="${base_y_size}" z="${base_z_size}" />
     </inertial>
     <visual>
       <origin xyz="0 0 0" rpy="0 0 ${M_PI/2}" />
       <geometry>
-        <mesh filename="package://am_description/urdf/am_chassis.stl" scale="0.001 0.001 0.001"/>
-        <box size="${base_x_size} ${base_y_size} ${base_z_size}"/>
+        <mesh filename="package://am_description/urdf/am_chassis.stl" scale="0.001 0.001 0.001" />
+        <box size="${base_x_size} ${base_y_size} ${base_z_size}" />
       </geometry>
       <material name="DarkGreen" />
@@ -42,5 +42,5 @@
       <origin xyz="0.17 0 0.08" rpy="0 0 0 " />
       <geometry>
-        <box size="0.65 0.50 0.20"/>
+        <box size="0.65 0.50 0.20" />
       </geometry>
     </collision>
@@ -51,31 +51,37 @@
   </gazebo>
   <!-- WHEELs -->
-  <wheel fb="back" lr="right" parent="base_link" translateY="-0.24" translateX="0.0" translateZ="0.0" wheel_radius="0.1225" wheel_height="0.032" flip="1"/>
-  <wheel fb="back" lr="left" parent="base_link" translateY="0.24" translateX="0.0" translateZ="0.0" wheel_radius="0.1225" wheel_height="0.032" flip="1"/>
+  <wheel fb="back" lr="right" parent="base_link" translateY="-0.24" translateX="0.0" translateZ="0.0"
+         wheel_radius="0.1225" wheel_height="0.032" flip="1" />
+  <wheel fb="back" lr="left" parent="base_link" translateY="0.24" translateX="0.0" translateZ="0.0"
+         wheel_radius="0.1225" wheel_height="0.032" flip="1" />
 <!--
-  <wheel fb="front" lr="right" parent="base_link" translateY="-0.15" translateX="0.35" translateZ="-0.065" wheel_radius="0.06" wheel_height="0.05" flip="1"/>
-  <wheel fb="front" lr="left" parent="base_link" translateY="0.15" translateX="0.35" translateZ="-0.065" wheel_radius="0.06" wheel_height="0.05" flip="1"/>
+  <wheel fb="front" lr="right" parent="base_link" translateY="-0.15" translateX="0.35" translateZ="-0.065"
+         wheel_radius="0.06" wheel_height="0.05" flip="1"/>
+  <wheel fb="front" lr="left" parent="base_link" translateY="0.15" translateX="0.35" translateZ="-0.065"
+         wheel_radius="0.06" wheel_height="0.05" flip="1"/>
 -->
-  <swivel_wheel fb="front" lr="right" parent="base_link" translateY="-0.16" translateX="0.355" translateZ="0.03" wheel_radius="0.05" wheel_height="0.05" flip="0"/>
-  <swivel_wheel fb="front" lr="left" parent="base_link" translateY="0.16" translateX="0.355" translateZ="0.03" wheel_radius="0.05" wheel_height="0.05" flip="0"/>
+  <swivel_wheel fb="front" lr="right" parent="base_link" translateY="-0.16" translateX="0.355" translateZ="0.03"
+                wheel_radius="0.05" wheel_height="0.05" flip="0" />
+  <swivel_wheel fb="front" lr="left" parent="base_link" translateY="0.16" translateX="0.355" translateZ="0.03"
+                wheel_radius="0.05" wheel_height="0.05" flip="0" />
   <!-- LOOP SENSORs -->
-  <sensorpos name="loop_front_center" parent="base_link" translateX="0.38" translateY="0.0" translateZ="-0.04"/>
-  <sensorpos name="loop_front_right" parent="base_link" translateX="0.38" translateY="-0.07" translateZ="-0.04"/>
-  <sensorpos name="loop_rear_left" parent="base_link" translateX="-0.07" translateY="0.14" translateZ="-0.04"/>
-  <sensorpos name="loop_rear_right" parent="base_link" translateX="-0.07" translateY="-0.14" translateZ="-0.04"/>
+  <sensorpos name="loop_front_center" parent="base_link" translateX="0.38" translateY="0.0" translateZ="-0.04" />
+  <sensorpos name="loop_front_right" parent="base_link" translateX="0.38" translateY="-0.07" translateZ="-0.04" />
+  <sensorpos name="loop_rear_left" parent="base_link" translateX="-0.07" translateY="0.14" translateZ="-0.04" />
+  <sensorpos name="loop_rear_right" parent="base_link" translateX="-0.07" translateY="-0.14" translateZ="-0.04" />
   <!-- CONFINEMENT SENSORs -->
-  <sensorpos name="col_front_chassis" parent="base_link" translateX="0.55" translateY="0.0" translateZ="0.00"/>
-  <sensorpos name="col_front_left" parent="base_link" translateX="0.43" translateY="0.24" translateZ="0.00"/>
-  <sensorpos name="col_front_right" parent="base_link" translateX="0.43" translateY="-0.24" translateZ="0.00"/>
-  <sensorpos name="col_rear_left" parent="base_link" translateX="-0.10" translateY="0.24" translateZ="0.0"/>
-  <sensorpos name="col_rear_right" parent="base_link" translateX="-0.10" translateY="-0.24" translateZ="0.0"/>
+  <sensorpos name="col_front_chassis" parent="base_link" translateX="0.55" translateY="0.0" translateZ="0.00" />
+  <sensorpos name="col_front_left" parent="base_link" translateX="0.43" translateY="0.24" translateZ="0.00" />
+  <sensorpos name="col_front_right" parent="base_link" translateX="0.43" translateY="-0.24" translateZ="0.00" />
+  <sensorpos name="col_rear_left" parent="base_link" translateX="-0.10" translateY="0.24" translateZ="0.0" />
+  <sensorpos name="col_rear_right" parent="base_link" translateX="-0.10" translateY="-0.24" translateZ="0.0" />
   <!-- CUTTING DISC -->
   <link name="cutting_disc_center">
     <visual>
-        <origin xyz="0 0 0" rpy="0 0 0" />
-        <geometry>
-            <cylinder length="0.01" radius="0.11" />
-        </geometry>
-        <material name="Purple" />
+      <origin xyz="0 0 0" rpy="0 0 0" />
+      <geometry>
+        <cylinder length="0.01" radius="0.11" />
+      </geometry>
+      <material name="Purple" />
     </visual>
   </link>
@@ -84,16 +90,16 @@
   </gazebo>
   <joint name="cutting_disc_center_joint" type="fixed">
-    <parent link="base_link"/>
+    <parent link="base_link" />
     <child link="cutting_disc_center" />
-	<origin xyz="0.25 0.0 -0.07" rpy="0 0 0" />
+    <origin xyz="0.25 0.0 -0.07" rpy="0 0 0" />
   </joint>
   <!-- Antenna -->
   <link name="antenna_center">
     <visual>
-        <origin xyz="0 0 0" rpy="0 0 0" />
-        <geometry>
-            <cylinder length="0.01" radius="0.05" />
-        </geometry>
-        <material name="Purple" />
+      <origin xyz="0 0 0" rpy="0 0 0" />
+      <geometry>
+        <cylinder length="0.01" radius="0.05" />
+      </geometry>
+      <material name="Purple" />
     </visual>
   </link>
@@ -102,7 +108,7 @@
   </gazebo>
   <joint name="antenna_center_joint" type="fixed">
-    <parent link="base_link"/>
+    <parent link="base_link" />
     <child link="antenna_center" />
-	<origin xyz="0.27 0.0 0.0" rpy="0 0 0" />
+    <origin xyz="0.27 0.0 0.0" rpy="0 0 0" />
   </joint>
   <!-- GAZEBO STUFF -->
@@ -125,57 +131,57 @@
     <plugin name="gazebo_ros_control" filename="libgazebo_ros_control.so" />
     <plugin name="imu_plugin" filename="libhector_gazebo_ros_imu.so">
-    <alwaysOn>true</alwaysOn>
-    <bodyName>base_link</bodyName>
-    <topicName>imu</topicName>
-    <serviceName>imu_service</serviceName>
-    <updateRate>100.0</updateRate>
-    <rpyOffsets>0 0 0</rpyOffsets> <!-- deprecated -->
+      <alwaysOn>true</alwaysOn>
+      <bodyName>base_link</bodyName>
+      <topicName>imu</topicName>
+      <serviceName>imu_service</serviceName>
+      <updateRate>100.0</updateRate>
+      <rpyOffsets>0 0 0</rpyOffsets> <!-- deprecated -->
 <!--
-	    <gaussianNoise>0.0</gaussianNoise>
-	    <accelDrift>0.5 0.5 0.5</accelDrift>
-	    <accelGaussianNoise>0.35 0.35 0.3</accelGaussianNoise>
-	    <rateDrift>0.1 0.1 0.1</rateDrift>
-	    <rateGaussianNoise>0.05 0.05 0.015</rateGaussianNoise>
-	    <headingDrift>0.1</headingDrift>
-	    <headingGaussianNoise>1.00</headingGaussianNoise>
+      <gaussianNoise>0.0</gaussianNoise>
+      <accelDrift>0.5 0.5 0.5</accelDrift>
+      <accelGaussianNoise>0.35 0.35 0.3</accelGaussianNoise>
+      <rateDrift>0.1 0.1 0.1</rateDrift>
+      <rateGaussianNoise>0.05 0.05 0.015</rateGaussianNoise>
+      <headingDrift>0.1</headingDrift>
+      <headingGaussianNoise>1.00</headingGaussianNoise>
 -->
-		<gaussianNoise>0.0</gaussianNoise>  <!-- deprecated -->
-	    <accelDrift>0.0 0.0 0.0</accelDrift>
-	    <accelGaussianNoise>0.0 0.0 0.0</accelGaussianNoise>
-	    <rateDrift>0.0 0.0 0.0</rateDrift>
-	    <rateGaussianNoise>0.0 0.0 0.0</rateGaussianNoise>
-	    <headingDrift>0.0</headingDrift>
-	    <headingGaussianNoise>0.00</headingGaussianNoise>
+      <gaussianNoise>0.0</gaussianNoise>  <!-- deprecated -->
+      <accelDrift>0.0 0.0 0.0</accelDrift>
+      <accelGaussianNoise>0.0 0.0 0.0</accelGaussianNoise>
+      <rateDrift>0.0 0.0 0.0</rateDrift>
+      <rateGaussianNoise>0.0 0.0 0.0</rateGaussianNoise>
+      <headingDrift>0.0</headingDrift>
+      <headingGaussianNoise>0.00</headingGaussianNoise>
     </plugin>
     <plugin name="am_gazebo_wheelencoder" filename="libam_gazebo_wheelencoder.so">
-	</plugin>
+    </plugin>
     <plugin name="automower_gps_sim" filename="libhector_gazebo_ros_gps.so">
-	  <alwaysOn>true</alwaysOn>
-	  <updateRate>4.0</updateRate>
-	  <bodyName>base_link</bodyName>
-	  <topicName>fix</topicName>
-	  <velocityTopicName>fix_vel</velocityTopicName>
-	  <drift>5.0 5.0 5.0</drift>
-	  <gaussianNoise>0.1 0.1 0.1</gaussianNoise>
-	  <velocityDrift>0 0 0</velocityDrift>
-	  <velocityGaussianNoise>0.1 0.1 0.1</velocityGaussianNoise>
+      <alwaysOn>true</alwaysOn>
+      <updateRate>4.0</updateRate>
+      <bodyName>base_link</bodyName>
+      <topicName>fix</topicName>
+      <velocityTopicName>fix_vel</velocityTopicName>
+      <drift>5.0 5.0 5.0</drift>
+      <gaussianNoise>0.1 0.1 0.1</gaussianNoise>
+      <velocityDrift>0 0 0</velocityDrift>
+      <velocityGaussianNoise>0.1 0.1 0.1</velocityGaussianNoise>
     </plugin>
   </gazebo>
   <gazebo reference="base_link">
-	<sensor name="automower_sensor" type="contact">
-		<always_on>true</always_on>
-		<update_rate>50</update_rate>
-		<contact>
-			<collision>base_link_collision</collision>
-		</contact>
-		<plugin name="automower_sensors_plugin" filename="libam_gazebo_sensors.so">
-			<always_on>true</always_on>
-			<update_rate>20</update_rate>
-			<bumperTopicName>sensor_status</bumperTopicName>
-			<loopTopicName>loop</loopTopicName>
-			<!-- 0x01 = FC, 0x02 = FR, 0x04 = RL, 0x08 = RR -->
-			<loopOutsideSensors>15</loopOutsideSensors>
-		</plugin>
-	</sensor>
+    <sensor name="automower_sensor" type="contact">
+      <always_on>true</always_on>
+      <update_rate>50</update_rate>
+      <contact>
+        <collision>base_link_collision</collision>
+      </contact>
+      <plugin name="automower_sensors_plugin" filename="libam_gazebo_sensors.so">
+        <always_on>true</always_on>
+        <update_rate>20</update_rate>
+        <bumperTopicName>sensor_status</bumperTopicName>
+        <loopTopicName>loop</loopTopicName>
+        <!-- 0x01 = FC, 0x02 = FR, 0x04 = RL, 0x08 = RR -->
+        <loopOutsideSensors>15</loopOutsideSensors>
+      </plugin>
+    </sensor>
   </gazebo>
 </robot>

File: am_description/urdf/materials.urdf.xacro (robot description, xacro)
@@ -2,32 +2,32 @@
 <robot>
   <material name="Black">
-    <color rgba="0.0 0.0 0.0 1.0"/>
+    <color rgba="0.0 0.0 0.0 1.0" />
   </material>
   <material name="Blue">
-    <color rgba="0.0 0.0 0.8 1.0"/>
+    <color rgba="0.0 0.0 0.8 1.0" />
   </material>
   <material name="Green">
-    <color rgba="0.0 0.1 0.0 1.0"/>
+    <color rgba="0.0 0.1 0.0 1.0" />
   </material>
   <material name="DarkGreen">
-    <color rgba="0.2 0.6 0.0 1.0"/>
+    <color rgba="0.2 0.6 0.0 1.0" />
   </material>
   <material name="Gray">
-    <color rgba="0.7 0.7 0.7 1.0"/>
+    <color rgba="0.7 0.7 0.7 1.0" />
   </material>
   <material name="DarkGray">
-    <color rgba="0.3 0.3 0.3 1.0"/>
+    <color rgba="0.3 0.3 0.3 1.0" />
   </material>
   <material name="Red">
-    <color rgba="0.8 0.0 0.0 1.0"/>
+    <color rgba="0.8 0.0 0.0 1.0" />
   </material>
   <material name="Purple">
-    <color rgba="1.0 0.0 1.0 1.0"/>
+    <color rgba="1.0 0.0 1.0 1.0" />
   </material>
   <material name="White">
-    <color rgba="1.0 1.0 1.0 1.0"/>
+    <color rgba="1.0 1.0 1.0 1.0" />
   </material>
   <material name="Yellow">
-    <color rgba="0.8 0.8 0.0 1.0"/>
+    <color rgba="0.8 0.8 0.0 1.0" />
   </material>
 </robot>

File: am_description/urdf/sensorpos.urdf.xacro (robot description, xacro)
@@ -1,15 +1,14 @@
 <?xml version="1.0"?>
 <robot name="sensorpos" xmlns:xacro="http://www.ros.org/wiki/xacro">
- <!-- NOTE! Must have a mass/inertial so that Gazebo does not ignore these... -->
+  <!-- NOTE! Must have a mass/inertial so that Gazebo does not ignore these... -->
   <xacro:macro name="sensorpos" params="name parent translateX translateY translateZ ">
     <link name="${name}">
-		<inertial>
-			<origin xyz="0 0 1" rpy="0 0 0"/>
-			<mass value="0.01"/>
-			<inertia
-				ixx="1.0" ixy="0.0" ixz="0.0"
-				iyy="1.0" iyz="0.0"
-				izz="1.0"/>
-		</inertial>
+      <inertial>
+        <origin xyz="0 0 1" rpy="0 0 0" />
+        <mass value="0.01" />
+        <inertia ixx="1.0" ixy="0.0" ixz="0.0"
+                 iyy="1.0" iyz="0.0"
+                 izz="1.0" />
+      </inertial>
     </link>
     <gazebo reference="${name}">
@@ -18,6 +17,6 @@
     </gazebo>
     <joint name="${name}_joint" type="continuous">
-      <parent link="${parent}"/>
-      <child link="${name}"/>
+      <parent link="${parent}" />
+      <child link="${name}" />
       <origin xyz="${translateX} ${translateY} ${translateZ}" rpy="0 0 0" />
     </joint>

File: am_description/urdf/swivel_wheel.urdf.xacro (robot description, xacro)
@@ -13,21 +13,21 @@
 -->
   <xacro:macro name="cylinder_inertia" params="m r h">
-    <inertia  ixx="${m*(3*r*r+h*h)/12}" ixy = "0" ixz = "0"
-              iyy="${m*(3*r*r+h*h)/12}" iyz = "0"
-              izz="${m*r*r/2}" />
+    <inertia ixx="${m*(3*r*r+h*h)/12}" ixy="0" ixz="0"
+             iyy="${m*(3*r*r+h*h)/12}" iyz="0"
+             izz="${m*r*r/2}" />
   </xacro:macro>
-  <xacro:macro name = "swivel_arm" params="lr index l offset">
+  <xacro:macro name="swivel_arm" params="lr index l offset">
     <link name="sw_arm_${lr}_${index}">
       <inertial>
         <mass value="0.01" />
         <origin xyz="0 0 0" />
-        <cylinder_inertia  m="0.01" r="0.004" h="${l}" />
+        <cylinder_inertia m="0.01" r="0.004" h="${l}" />
       </inertial>
       <visual>
         <geometry>
-        <cylinder radius="0.004" length="${l}"/>
+          <cylinder radius="0.004" length="${l}" />
         </geometry>
         <material name="silver">
-         <color rgba="0.3 0.3 0.3 1"/>
+          <color rgba="0.3 0.3 0.3 1" />
         </material>
         <origin rpy="0 0 0" xyz="${offset}" />
@@ -35,35 +35,36 @@
     </link>
   </xacro:macro>
-  <xacro:macro name="swivel_wheel" params="fb lr parent translateX translateY translateZ wheel_radius wheel_height flip"> <!--fb : front, back ; lr: left, right -->
+  <xacro:macro name="swivel_wheel"
+               params="fb lr parent translateX translateY translateZ wheel_radius wheel_height flip"> <!--fb : front, back ; lr: left, right -->
     <!-- First link connected to parent-->
-    <swivel_arm lr = "${lr}" index = "1" l = "0.06" offset="0 0 -0.03"/>
+    <swivel_arm lr="${lr}" index="1" l="0.06" offset="0 0 -0.03" />
     <joint name="sw_arm_${lr}_connect_1" type="continuous">
       <origin xyz="${translateX} ${translateY} ${translateZ}" rpy="0 0 0" />
       <axis xyz="0 0 1" rpy="0 0 0" />
-      <parent link="${parent}"/>
-      <child link="sw_arm_${lr}_1"/>
-      <limit effort="100" velocity="100"/>
-      <joint_properties damping="0.0" friction="0.0"/>
+      <parent link="${parent}" />
+      <child link="sw_arm_${lr}_1" />
+      <limit effort="100" velocity="100" />
+      <joint_properties damping="0.0" friction="0.0" />
     </joint>
     <!-- Second link connected to first-->
-    <swivel_arm lr = "${lr}" index = "2" l = "0.04" offset="0 0 0.02"/>
+    <swivel_arm lr="${lr}" index="2" l="0.04" offset="0 0 0.02" />
     <joint name="sw_arm_${lr}_connect_2" type="fixed">
       <origin rpy="1.5707 0 0" xyz="0 0 -0.06" />
-      <parent link="sw_arm_${lr}_1"/>
-      <child link="sw_arm_${lr}_2"/>
+      <parent link="sw_arm_${lr}_1" />
+      <child link="sw_arm_${lr}_2" />
     </joint>
     <!-- Third link connected to second-->
-    <swivel_arm lr = "${lr}" index = "3" l = "0.06" offset="0 0 -0.03"/>
+    <swivel_arm lr="${lr}" index="3" l="0.06" offset="0 0 -0.03" />
     <joint name="sw_arm_${lr}_connect_3" type="fixed">
       <origin rpy="-1.5707 0 -0.78" xyz="0 0 0.04" />
-      <parent link="sw_arm_${lr}_2"/>
-      <child link="sw_arm_${lr}_3"/>
+      <parent link="sw_arm_${lr}_2" />
+      <child link="sw_arm_${lr}_3" />
     </joint>
     <!-- Fourth link connected to third-->
-    <swivel_arm lr = "${lr}" index = "4" l = "0.04" offset="0 0 -0.02"/>
+    <swivel_arm lr="${lr}" index="4" l="0.04" offset="0 0 -0.02" />
     <joint name="sw_arm_${lr}_connect_4" type="fixed">
       <origin rpy="1.5707 0 0" xyz="0 0 -0.060" />
-      <parent link="sw_arm_${lr}_3"/>
-      <child link="sw_arm_${lr}_4"/>
+      <parent link="sw_arm_${lr}_3" />
+      <child link="sw_arm_${lr}_4" />
     </joint>
     <!-- Wheel connected to fourth-->
@@ -85,23 +86,23 @@
         <mass value="${wheel_mass}" />
         <origin xyz="0 0 0" />
-        <cylinder_inertia  m="${wheel_mass}" r="${wheel_radius}" h="${wheel_height}" />
+        <cylinder_inertia m="${wheel_mass}" r="${wheel_radius}" h="${wheel_height}" />
       </inertial>
     </link>
     <gazebo reference="${fb}_${lr}_swivel_wheel">
-      <mu1 value="0.8"/>
-      <mu2 value="0.8"/>
-      <kp  value="10000000.0" />
-      <kd  value="1.0" />
-      <fdir1 value="1 0 0"/>
+      <mu1 value="0.8" />
+      <mu2 value="0.8" />
+      <kp value="10000000.0" />
+      <kd value="1.0" />
+      <fdir1 value="1 0 0" />
       <material>Gazebo/Black</material>
       <turnGravityOff>false</turnGravityOff>
     </gazebo>
     <joint name="${fb}_${lr}_swivel_wheel_joint" type="continuous">
-      <parent link="sw_arm_${lr}_4"/>
-      <child link="${fb}_${lr}_swivel_wheel"/>
+      <parent link="sw_arm_${lr}_4" />
+      <child link="${fb}_${lr}_swivel_wheel" />
       <origin rpy="0 0 0" xyz="0 0 -0.04" />
       <axis xyz="0 0 1" rpy="0 0 0" />
-      <limit effort="100" velocity="100"/>
-      <joint_properties damping="0.0" friction="0.0"/>
+      <limit effort="100" velocity="100" />
+      <joint_properties damping="0.0" friction="0.0" />
     </joint>
     <!-- Transmission is important to link the joints and the controller -->

File: am_description/urdf/wheel.urdf.xacro (robot description, xacro)
@@ -13,9 +13,10 @@
 -->
   <xacro:macro name="cylinder_inertia" params="m r h">
-    <inertia  ixx="${m*(3*r*r+h*h)/12}" ixy = "0" ixz = "0"
-              iyy="${m*(3*r*r+h*h)/12}" iyz = "0"
-              izz="${m*r*r/2}" />
+    <inertia ixx="${m*(3*r*r+h*h)/12}" ixy="0" ixz="0"
+             iyy="${m*(3*r*r+h*h)/12}" iyz="0"
+             izz="${m*r*r/2}" />
   </xacro:macro>
-  <xacro:macro name="wheel" params="fb lr parent translateX translateY translateZ wheel_radius wheel_height flip"> <!--fb : front, back ; lr: left, right -->
+  <xacro:macro name="wheel"
+               params="fb lr parent translateX translateY translateZ wheel_radius wheel_height flip"> <!--fb : front, back ; lr: left, right -->
     <link name="${fb}_${lr}_wheel">
       <visual>
@@ -36,23 +37,23 @@
         <!-- <origin xyz="0 0 0" rpy="${flip*M_PI/2} 0 0"/> -->
         <origin xyz="0 0 0" />
-        <cylinder_inertia  m="${wheel_mass}" r="${wheel_radius}" h="${wheel_height}" />
+        <cylinder_inertia m="${wheel_mass}" r="${wheel_radius}" h="${wheel_height}" />
       </inertial>
     </link>
     <gazebo reference="${fb}_${lr}_wheel">
-      <mu1 value="100.0"/>
-      <mu2 value="100.0"/>
-      <kp  value="10000000.0" />
-      <kd  value="1.0" />
-      <fdir1 value="1 0 0"/>
+      <mu1 value="100.0" />
+      <mu2 value="100.0" />
+      <kp value="10000000.0" />
+      <kd value="1.0" />
+      <fdir1 value="1 0 0" />
       <material>Gazebo/Black</material>
       <turnGravityOff>false</turnGravityOff>
     </gazebo>
     <joint name="${fb}_${lr}_wheel_joint" type="continuous">
-      <parent link="${parent}"/>
-      <child link="${fb}_${lr}_wheel"/>
+      <parent link="${parent}" />
+      <child link="${fb}_${lr}_wheel" />
       <origin xyz="${translateX} ${translateY} ${translateZ}" rpy="0 0 0" />
       <axis xyz="0 1 0" rpy="0 0 0" />
-      <limit effort="1000" velocity="100"/>
-      <joint_properties damping="0.0" friction="0.0"/>
+      <limit effort="1000" velocity="100" />
+      <joint_properties damping="0.0" friction="0.0" />
     </joint>
     <!-- Transmission is important to link the joints and the controller -->
